File: SCH-PCB/ShieldRelay/shieldRelay.brd (EAGLE design)
At the start: 160 x 100 mm, 3 parts

Commit message: update
Parts:
- removed U$1: NANO, Arduino-clone:NANO
- added C16: KAF21KR71H225KU, KAF21KR71H225KU:CAPC2012X140N
- added C17: EEH-ZU1V681UP, EEH-ZU1V681UP:EEHZS1H221P
- added C3: 220uf 25V, MAL203836221E3:CAPPRD350W60D850H1250
- added D1, D2, D3, D4, D5: FM4004-W, FM4004-W:DIONM5025X231N
- added D8: B340A-13-F, B340A-13-F:DIOM5226X240N
- added FB1: BLM21PG221SN1D, BLM21PG221SN1D:BEADC2012X105N
- added H1, H2, H3, H4: 3MM_HOLE, 3mm_special_hole:3MM_HOLE
- added IC1: LM2596SX-5.0_NOPB, LM2596SX-5.0_NOPB:KTT0005B
- added JP1, JP2, JP3, JP4, JP5, JP6: (no value), pinhead:1X15
- added JP10, JP8, JP9: (no value), pinhead:2X04
- added JP7: (no value), pinhead:1X03
- added K1: SLA-05VDC-SL-C, SLA-05VDC-SL-C:SLA05VDCSLC
- added K2, K6: SRD-05VDC-SL-C, SRD-05VDC-SL-C:SRD05VDCSLC
- added K3, K5: G3MB-202PL-DC5, G3MB-202PL-DC5:G3MB202PLDC5
- added L1: 33uh 12x12, 744770133:WE-PD_1260/1245/1280/121054
- added LED1, LED2, LED3, LED4, LED6: 150080SS75000, SamacSys_Parts:LEDC2012X80N
- added Q1, Q2, Q3, Q4, Q5: MMST2222A-7-F, MMST2222A-7-F:SOT65P210X110-3N
- added R1, R10, R2, R3, R4, R5, R6, R7, R8, R9: 1k, ERA-3AED102V:ERA3AEB101V
- added RELAY_CONTROL: (no value), pinhead:2X05
- moved BOARD1 54.9 mm to (150.6, 18.8), turned to 90 degrees
- moved NODE1 50.4 mm to (179.3, 25.1), turned to 180 degrees
Connections:
- new net +3V3: JP7.3
- new net +5V: C3.1, D1.1, D2.1, D3.1, D4.1, D5.1, IC1.4, JP7.1, K1.5, K2.1, K3.3, K5.3, K6.1, L1.2, R1.2, R3.2, R5.2, R7.2, R9.2
- new net IN1: R6.2, RELAY_CONTROL.1
- new net IN2: R2.2, RELAY_CONTROL.3
- new net IN3: R4.2, RELAY_CONTROL.5
- new net IN4: R8.2, RELAY_CONTROL.7
- new net IN5: R10.2, RELAY_CONTROL.9
- new net N$1: LED1.2, R3.1
- new net N$10: LED3.2, R7.1
- new net N$11: D4.2, K5.4, LED3.1, Q4.2
- new net N$12: Q4.1, R8.1
- new net N$13: LED4.2, R9.1
- new net N$14: D5.2, K3.4, LED4.1, Q5.2
- new net N$15: Q5.1, R10.1
- new net N$16: BOARD1.3V3
- new net N$17: JP1.1, JP2.1
- new net N$18: D8.1, IC1.2, L1.1
- new net N$19: JP1.2, JP2.2
- new net N$2: LED6.2, R1.1
- new net N$20: JP1.3, JP2.3
- new net N$21: JP1.4, JP2.4
- new net N$22: JP1.5, JP2.5
- new net N$23: RELAY_CONTROL.10
- new net N$24: RELAY_CONTROL.8
- new net N$25: RELAY_CONTROL.6
- new net N$26: RELAY_CONTROL.4
- new net N$27: RELAY_CONTROL.2
- new net N$28: JP1.6, JP2.6
- new net N$29: JP1.7, JP2.7
- new net N$3: D1.2, K2.4, LED6.1, Q1.2
- new net N$30: JP1.8, JP2.8
- new net N$31: JP1.9, JP2.9
- new net N$32: JP1.10, JP2.10
- new net N$33: JP1.11, JP2.11
- new net N$34: JP1.12, JP2.12
- new net N$35: JP1.13, JP2.13
- new net N$36: JP1.14, JP2.14
- new net N$37: JP1.15, JP2.15
- new net N$38: BOARD1.GND@1
- new net N$39: JP3.1, JP3.10, JP3.11, JP3.12, JP3.13, JP3.14, JP3.15, JP3.2, JP3.3, JP3.4, JP3.5, JP3.6, JP3.7, JP3.8, JP3.9, JP4.1, JP4.10, JP4.11, JP4.12, JP4.13, JP4.14, JP4.15, JP4.2, JP4.3, JP4.4, JP4.5, JP4.6, JP4.7, JP4.8, JP4.9, JP7.2, JP8.1, JP8.2, JP8.3, JP8.4, JP8.5, JP8.6, JP8.7, JP8.8
- new net N$4: Q1.1, R2.1
- new net N$40: BOARD1.D15
- new net N$41: BOARD1.D2
- new net N$42: BOARD1.D4
- new net N$43: BOARD1.D16
- new net N$44: BOARD1.D17
- new net N$45: BOARD1.D5
- new net N$46: BOARD1.D18
- new net N$47: BOARD1.D19
- new net N$48: BOARD1.D21
- new net N$49: BOARD1.D3
- new net N$5: D2.2, K6.4, LED1.1, Q2.2
- new net N$50: BOARD1.D1
- new net N$51: BOARD1.D22
- new net N$52: BOARD1.D23
- new net N$53: BOARD1.EN
- new net N$54: BOARD1.VP
- new net N$55: BOARD1.VN
- new net N$56: BOARD1.D34
- new net N$57: BOARD1.D35
- new net N$58: BOARD1.D32
- new net N$59: BOARD1.D33
- new net N$6: Q2.1, R4.1
- new net N$60: BOARD1.D25
- new net N$61: BOARD1.D26
- new net N$62: BOARD1.D27
- new net N$63: BOARD1.D14
- new net N$64: BOARD1.D12
- new net N$65: BOARD1.D13
- new net N$66: BOARD1.GND
- new net N$67: BOARD1.VIN
- new net N$7: LED2.2, R5.1
- new net N$8: D3.2, K1.6, LED2.1, Q3.2
- new net N$9: Q3.1, R6.1
- new net VCC: FB1.2
- new net VCC/2: C16.1, C17.1, FB1.1, IC1.1, JP10.1, JP10.2, JP10.3, JP10.4, JP10.5, JP10.6, JP10.7, JP10.8
- net GND: now also C16.2, C17.2, C3.2, D8.2, IC1.3, IC1.5, IC1.6, JP5.1, JP5.10, JP5.11, JP5.12, JP5.13, JP5.14, JP5.15, JP5.2, JP5.3, JP5.4, JP5.5, JP5.6, JP5.7, JP5.8, JP5.9, JP6.1, JP6.10, JP6.11, JP6.12, JP6.13, JP6.14, JP6.15, JP6.2, JP6.3, JP6.4, JP6.5, JP6.6, JP6.7, JP6.8, JP6.9, JP9.1, JP9.2, JP9.3, JP9.4, JP9.5, JP9.6, JP9.7, JP9.8, Q1.3, Q2.3, Q3.3, Q4.3, Q5.3
Other:
- board size 160 x 100 mm -> 99 x 100 mm

Commit message: FEAT: update library esp32 and remove nodemcu v2
Parts:
- moved NODE1 336.3 mm to (21.8, -272.0), turned to 0 degrees
- moved BOARD1 324.0 mm to (-24.1, -254.0), turned to 270 degrees
Changed lines of the file:
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@@
 </autorouter>
 <elements>
-<element name="BOARD1" library="ESP32-DEVKITV1" package="ESP32-DEVKITV1" value="ESP32DEVKITV1" x="150.622" y="18.796" smashed="yes" rot="R90">
-<attribute name="ESP32-DEVKITV1" value="" x="155.702" y="74.676" size="1.778" layer="27" rot="R90" display="off"/>
-<attribute name="NAME" x="144.002" y="19.146" size="1.27" layer="21" rot="R90"/>
-</element>
-<element name="NODE1" library="nodemcu_esp8266" package="NODEMCU_ESP8266" value="NODEMCU_ESP8266" x="179.324" y="25.146" smashed="yes" rot="R180">
-<attribute name="NAME" x="190.754" y="-2.794" size="1.27" layer="25" rot="R180"/>
-<attribute name="VALUE" x="190.754" y="51.816" size="1.27" layer="27" rot="R180"/>
+<element name="BOARD1" library="ESP32-DEVKITV1" package="ESP32-DEVKITV1" value="ESP32DEVKITV1" x="-24.13" y="-254" smashed="yes" rot="R270">
+<attribute name="ESP32-DEVKITV1" value="" x="-29.21" y="-309.88" size="1.778" layer="27" rot="R270" display="off"/>
+<attribute name="NAME" x="-17.51" y="-254.35" size="1.27" layer="21" rot="R270"/>
+</element>
+<element name="NODE1" library="nodemcu_esp8266" package="NODEMCU_ESP8266" value="NODEMCU_ESP8266" x="21.844" y="-272.034" smashed="yes">
+<attribute name="NAME" x="10.414" y="-244.094" size="1.27" layer="25"/>
+<attribute name="VALUE" x="10.414" y="-298.704" size="1.27" layer="27"/>
 </element>
 <element name="K1" library="SLA-05VDC-SL-C" package="SLA05VDCSLC" value="SLA-05VDC-SL-C" x="39.116" y="81.788" smashed="yes" rot="R90">
@@
 <signals>
 <signal name="3V3">
+<wire x1="190.754" y1="6.096" x2="167.894" y2="16.256" width="0" layer="19" extent="1-1"/>
+<wire x1="190.754" y1="28.956" x2="190.754" y2="6.096" width="0" layer="19" extent="1-1"/>
 <contactref element="NODE1" pad="3V3@1"/>
 <contactref element="NODE1" pad="3V3@2"/>
 <contactref element="NODE1" pad="3V3@3"/>
-<wire x1="190.754" y1="6.096" x2="167.894" y2="16.256" width="0" layer="19" extent="1-1"/>
-<wire x1="190.754" y1="28.956" x2="190.754" y2="6.096" width="0" layer="19" extent="1-1"/>
 </signal>
 <signal name="GND">
-<contactref element="NODE1" pad="GND@1"/>
-<contactref element="NODE1" pad="GND@2"/>
-<contactref element="NODE1" pad="GND@4"/>
-<contactref element="NODE1" pad="GND@3"/>
 <contactref element="Q1" pad="3"/>
 <contactref element="Q2" pad="3"/>
@@
 <wire x1="167.894" y1="8.636" x2="190.754" y2="8.636" width="0" layer="19" extent="1-1"/>
 <wire x1="167.894" y1="18.796" x2="167.894" y2="8.636" width="0" layer="19" extent="1-1"/>
+<contactref element="NODE1" pad="GND@1"/>
+<contactref element="NODE1" pad="GND@2"/>
+<contactref element="NODE1" pad="GND@4"/>
+<contactref element="NODE1" pad="GND@3"/>
 </signal>
 <signal name="VIN">

Commit message: FEAT: Positioning component
Parts:
- removed NODE1: NODEMCU_ESP8266, nodemcu_esp8266:NODEMCU_ESP8266
- added INPUT: 1759017, 1759017:SHDRRA2W103P0X508_1X2_1016X120
- moved JP10 325.3 mm to (51.3, 78.5)
- moved BOARD1 307.1 mm to (85.1, 33.0), turned to 90 degrees
- moved JP6 277.1 mm to (96.3, 50.8), turned to 90 degrees
- moved JP9 265.3 mm to (52.1, 24.9)
- moved JP4 264.1 mm to (93.5, 50.8), turned to 90 degrees
- moved JP5 260.6 mm to (48.8, 51.1), turned to 90 degrees
- moved JP7 260.1 mm to (43.4, 36.3), turned to 90 degrees
- moved JP8 255.7 mm to (41.4, 24.8)
- moved JP3 248.4 mm to (51.6, 51.1), turned to 90 degrees
- moved JP1 245.1 mm to (90.7, 50.8), turned to 90 degrees
- moved JP2 242.6 mm to (54.4, 51.1), turned to 90 degrees
- moved R9 232.2 mm to (44.7, 57.9)
- moved LED4 228.0 mm to (41.1, 57.9)
- moved RELAY_CONTROL 226.7 mm to (41.9, 47.5), turned to 270 degrees
- moved R10 215.0 mm to (36.3, 47.0)
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Connections:
- removed net 3V3: NODE1.3V3@1, NODE1.3V3@2, NODE1.3V3@3
- removed net VIN: NODE1.VIN
- net GND: now also INPUT.2; no longer NODE1.GND@1, NODE1.GND@2, NODE1.GND@3, NODE1.GND@4
- net VCC: now also INPUT.1
Other:
- board size 99 x 100 mm -> 99 x 78.9 mm

Commit message: FEAT: update library pinhead
Parts:
- added JP11, JP12: (no value), pinhead_mod:1X15
- JP1, JP2, JP3, JP4, JP5, JP6: device pinhead:1X15 -> pinhead_mod:1X15
- moved JP6 47.0 mm to (49.3, 50.8), turned to 270 degrees
- moved JP5 46.7 mm to (95.5, 50.8), flipped to the bottom, turned to 270 degrees
- moved C16 5.79 mm to (80.3, 83.6)
- moved FB1 5.79 mm to (82.0, 83.6)
- moved INPUT 2.84 mm to (87.4, 89.9)
- moved C17 0.76 mm to (91.4, 82.0)
- moved JP4 0.51 mm to (93.0, 50.8)
- moved JP3 0.36 mm to (51.8, 50.8), turned to 270 degrees
- moved JP2 0.25 mm to (54.4, 50.8)
- moved JP1 0.25 mm to (90.4, 50.8)
Connections:
- net N$17: now also JP11.1, JP12.1
- net N$19: now also JP11.2, JP12.2
- net N$20: now also JP11.3, JP12.3
- net N$21: now also JP11.4, JP12.4
- net N$22: now also JP11.5, JP12.5
- net N$28: now also JP11.6, JP12.6
- net N$29: now also JP11.7, JP12.7
- net N$30: now also JP11.8, JP12.8
- net N$31: now also JP11.9, JP12.9
- net N$32: now also JP11.10, JP12.10
- net N$33: now also JP11.11, JP12.11
- net N$34: now also JP11.12, JP12.12
- net N$35: now also JP11.13, JP12.13
- net N$36: now also JP11.14, JP12.14
- net N$37: now also JP11.15, JP12.15
